Commit message: feat: update link6 7 8

File: urdfs/ic_arm_with_wrist/urdf/ic_arm_with_wrist.urdf (robot description, URDF)
Before this commit: robot ic_arm_with_wrist, 9 links, 8 joints
Links:
- link link6: mass 0.880428 -> 0.920428
- link link7: mass 0.278311513027483 -> 0.408311513027483

Commit message: feat: the gc with wrist is almost ok

File: urdfs/ic_arm_with_wrist/urdf/ic_arm_with_wrist.urdf (robot description, URDF)
Before this commit: robot ic_arm_with_wrist, 9 links, 8 joints
Links:
- link base_link: geometry collision mesh filename=package://ic_arm_cnc/meshes/base_link.STL; visual mesh filename=package://ic_arm_cnc/meshes/base_link.STL
- link link1: mass 1.1167 -> 1.2167; geometry collision mesh filename=package://ic_arm_cnc/meshes/link1.STL; visual mesh filename=package://ic_arm_cnc/meshes/link1.STL
- link link2: mass 1.201 -> 1.301; geometry collision mesh filename=package://ic_arm_cnc/meshes/link2.STL; visual mesh filename=package://ic_arm_cnc/meshes/link2.STL
- link link3: mass 0.610 -> 0.710; geometry collision mesh filename=package://ic_arm_cnc/meshes/link3.STL; visual mesh filename=package://ic_arm_cnc/meshes/link3.STL
- link link4: geometry collision mesh filename=package://ic_arm_cnc/meshes/link4.STL; visual mesh filename=package://ic_arm_cnc/meshes/link4.STL
- link link5: geometry collision mesh filename=package://ic_arm_cnc/meshes/link5.STL; visual mesh filename=package://ic_arm_cnc/meshes/link5.STL
- link link6: mass 0.920428 -> 0.880428
- link link7: mass 0.408311513027483 -> 0.278311513027483
Joints:
- joint j1: axis 0 0 -1 -> 0 0 1
- joint j4: axis 0 0 -1 -> 0 0 1
