Commit message: feat: update urdf for now state

File: urdfs/ic_arm/urdf/ic_arm_cnc.urdf (robot description, URDF)
Before this commit: robot ic_arm_cnc, 7 links, 6 joints
Joints:
- joint j3: axis 0 0 -1 -> 0 0 1

File: urdfs/ic_arm_with_wrist/urdf/ic_arm_with_wrist.urdf (robot description, URDF)
Before this commit: robot ic_arm_with_wrist, 9 links, 8 joints
Joints:
- joint j3: axis 0 0 -1 -> 0 0 1
